File: Productivity Macro.sch (KiCad schematic (older format))
At the start: 34 parts, among them SW1 SW_Push, SW2 Rotary_Encoder_Switch, SW3 Rotary_Encoder_Switch, U1 ATmega32U4-AU, Y1 16Mhz

Commit message: klfg;;fkdlgdfgkl;kdfgl;
Parts:
- R1, R2, R3, R4: footprint (none) -> Resistor_SMD:R_0805_2012Metric
- SW2, SW3: footprint (none) -> Rotary_Encoder:RotaryEncoder_Alps_EC11E-Switch_Vertical_H20mm
- U1: footprint Package_QFP:TQFP-44_10x10mm_P0.8mm -> random-keyboard-parts:Molex-0548190589
- Y1: footprint (none) -> Crystal:Crystal_SMD_3225-4Pin_3.2x2.5mm
Changed lines of the file:
@@
 F 0 "R4" V 5104 3500 50  0000 C CNN
 F 1 "10K" V 5195 3500 50  0000 C CNN
-F 2 "" H 5300 3500 50  0001 C CNN
+F 2 "Resistor_SMD:R_0805_2012Metric" H 5300 3500 50  0001 C CNN
 F 3 "~" H 5300 3500 50  0001 C CNN
 	1    5300 3500
@@
 F 0 "U1" H 4300 1011 50  0000 C CNN
 F 1 "ATmega32U4-AU" H 4300 920 50  0000 C CNN
-F 2 "Package_QFP:TQFP-44_10x10mm_P0.8mm" H 4300 2900 50  0001 C CIN
+F 2 "random-keyboard-parts:Molex-0548190589" H 4300 2900 50  0001 C CIN
 F 3 "http://ww1.microchip.com/downloads/en/DeviceDoc/Atmel-7766-8-bit-AVR-ATmega16U4-32U4_Datasheet.pdf" H 4300 2900 50  0001 C CNN
 	1    4300 2900
@@
 F 0 "R2" V 2954 2400 50  0000 C CNN
 F 1 "22" V 3045 2400 50  0000 C CNN
-F 2 "" H 3150 2400 50  0001 C CNN
+F 2 "Resistor_SMD:R_0805_2012Metric" H 3150 2400 50  0001 C CNN
 F 3 "~" H 3150 2400 50  0001 C CNN
 	1    3150 2400
@@
 F 0 "R3" V 2604 2500 50  0000 C CNN
 F 1 "22" V 2695 2500 50  0000 C CNN
-F 2 "" H 2800 2500 50  0001 C CNN
+F 2 "Resistor_SMD:R_0805_2012Metric" H 2800 2500 50  0001 C CNN
 F 3 "~" H 2800 2500 50  0001 C CNN
 	1    2800 2500
@@
 F 0 "R1" H 3759 1146 50  0000 L CNN
 F 1 "R_Small" H 3759 1055 50  0000 L CNN
-F 2 "" H 3700 1100 50  0001 C CNN
+F 2 "Resistor_SMD:R_0805_2012Metric" H 3700 1100 50  0001 C CNN
 F 3 "~" H 3700 1100 50  0001 C CNN
 	1    3700 1100
@@
 F 0 "Y1" V 3254 1844 50  0000 L CNN
 F 1 "16Mhz" V 3345 1844 50  0000 L CNN
-F 2 "" H 3300 1700 50  0001 C CNN
+F 2 "Crystal:Crystal_SMD_3225-4Pin_3.2x2.5mm" H 3300 1700 50  0001 C CNN
 F 3 "~" H 3300 1700 50  0001 C CNN
 	1    3300 1700
@@
 F 0 "SW2" V 7454 1980 50  0000 L CNN
 F 1 "Rotary_Encoder_Switch" V 7545 1980 50  0000 L CNN
-F 2 "" H 7350 1910 50  0001 C CNN
+F 2 "Rotary_Encoder:RotaryEncoder_Alps_EC11E-Switch_Vertical_H20mm" H 7350 1910 50  0001 C CNN
 F 3 "~" H 7500 2010 50  0001 C CNN
 	1    7500 1750
@@
 F 0 "SW3" V 8954 1980 50  0000 L CNN
 F 1 "Rotary_Encoder_Switch" V 9045 1980 50  0000 L CNN
-F 2 "" H 8850 1910 50  0001 C CNN
+F 2 "Rotary_Encoder:RotaryEncoder_Alps_EC11E-Switch_Vertical_H20mm" H 8850 1910 50  0001 C CNN
 F 3 "~" H 9000 2010 50  0001 C CNN
 	1    9000 1750
