File: Productivity Macro.sch (KiCad schematic (older format))
At the start: 34 parts, among them SW1 SW_Push, SW2 Rotary_Encoder_Switch, SW3 Rotary_Encoder_Switch, U1 ATmega32U4-AU, Y1 16Mhz

Commit message: close
Parts:
- R1: value R_Small -> 10k
Connections:
- net COL0: now also U1.39 (PF4)
- net COL1: now also U1.38 (PF5)
- net COL2: now also U1.37 (PF6)
- net GND: now also USB1.6 (SHIELD)
- net ROW0: now also U1.22 (PD5)
- net ROW1: now also U1.29 (PB5)
- net ROW2: now also U1.26 (PD6)
- net PINB: now reaches U1.10 (PB2)
- net PINB: now also SW2.B
- net PINA: now reaches U1.11 (PB3)
- net PINA: now also SW2.A
- net PINA1: now reaches U1.36 (PF7)
- net PINA1: now also SW3.A
- net PINB1: now reaches U1.40 (PF1)
- net PINB1: now also SW3.B
Changed lines of the file:
@@
 P 3700 1100
 F 0 "R1" H 3759 1146 50  0000 L CNN
-F 1 "R_Small" H 3759 1055 50  0000 L CNN
+F 1 "10k" H 3759 1055 50  0000 L CNN
 F 2 "Resistor_SMD:R_0805_2012Metric" H 3700 1100 50  0001 C CNN
 F 3 "~" H 3700 1100 50  0001 C CNN
@@
 	0    -1   -1   0
 $EndComp
+Text GLabel 4900 4000 2    50   Input ~ 0
+COL0
+Text GLabel 4900 3100 2    50   Input ~ 0
+ROW0
+Text GLabel 4900 1900 2    50   Input ~ 0
+ROW1
+Text GLabel 4900 4100 2    50   Input ~ 0
+COL1
+Text GLabel 4900 4200 2    50   Input ~ 0
+COL2
+Text GLabel 4900 3200 2    50   Input ~ 0
+ROW2
+Text GLabel 4900 1700 2    50   Input ~ 0
+PINA
+Text GLabel 4900 1600 2    50   Input ~ 0
+PINB
+Text GLabel 7600 1450 1    50   Input ~ 0
+PINA
+Text GLabel 7400 1450 1    50   Input ~ 0
+PINB
+Text GLabel 4900 4300 2    50   Input ~ 0
+PINA1
+Text GLabel 4900 3900 2    50   Input ~ 0
+PINB1
+Text GLabel 8900 1450 1    50   Input ~ 0
+PINB1
+Text GLabel 9100 1450 1    50   Input ~ 0
+PINA1
+$Comp
+L power:GND #PWR0116
+U 1 1 6088BDB9
+P 6050 1450
+F 0 "#PWR0116" H 6050 1200 50  0001 C CNN
+F 1 "GND" H 6055 1277 50  0000 C CNN
+F 2 "" H 6050 1450 50  0001 C CNN
+F 3 "" H 6050 1450 50  0001 C CNN
+	1    6050 1450
+	1    0    0    -1
+$EndComp
 $EndSCHEMATC

Commit message: The beginning of the trackball
Parts:
- added J4: Conn_02x04_Counter_Clockwise, Connector_PinSocket_2.00mm:PinSocket_2x04_P2.00mm_Vertical, symbol Connector_Generic:Conn_02x04_Counter_Clockwise
Connections:
- net GND: now also J4.3 (Pin_3)
- net PINA: now also U1.9 (PB1); no longer U1.11 (PB3)
- net PINB: now also U1.8 (PB0); no longer U1.10 (PB2)
- net VCC: now also J4.8 (Pin_8)
- net ss: now reaches U1.12 (PB7)
- net ss: now also J4.1 (Pin_1)
- net mosi: now reaches U1.18 (PD0)
- net mosi: now also J4.6 (Pin_6)
- new net miso: J4.7 (Pin_7), U1.11 (PB3)
- new net motion: J4.2 (Pin_2)
- new net sclk: J4.5 (Pin_5), U1.10 (PB2)
Changed lines of the file:
@@
 Text GLabel 4900 3200 2    50   Input ~ 0
 ROW2
-Text GLabel 4900 1700 2    50   Input ~ 0
+Text GLabel 4900 1500 2    50   Input ~ 0
 PINA
-Text GLabel 4900 1600 2    50   Input ~ 0
+Text GLabel 4900 1400 2    50   Input ~ 0
 PINB
 Text GLabel 7600 1450 1    50   Input ~ 0
@@
 	1    0    0    -1
 $EndComp
+$Comp
+L Connector_Generic:Conn_02x04_Counter_Clockwise J4
+U 1 1 60BB48DB
+P 6300 4500
+F 0 "J4" H 6350 4817 50  0000 C CNN
+F 1 "Conn_02x04_Counter_Clockwise" H 6350 4726 50  0000 C CNN
+F 2 "Connector_PinSocket_2.00mm:PinSocket_2x04_P2.00mm_Vertical" H 6300 4500 50  0001 C CNN
+F 3 "~" H 6300 4500 50  0001 C CNN
+	1    6300 4500
+	1    0    0    -1
+$EndComp
+Text GLabel 6100 4400 0    50   Input ~ 0
+ss
+Text GLabel 6100 4500 0    50   Input ~ 0
+motion
+Text GLabel 6600 4500 2    50   Input ~ 0
+miso
+Text GLabel 6600 4600 2    50   Input ~ 0
+mosi
+Text GLabel 6600 4700 2    50   Input ~ 0
+sclk
+$Comp
+L power:GND #PWR0117
+U 1 1 60BB7D4F
+P 6100 4600
+F 0 "#PWR0117" H 6100 4350 50  0001 C CNN
+F 1 "GND" V 6105 4472 50  0000 R CNN
+F 2 "" H 6100 4600 50  0001 C CNN
+F 3 "" H 6100 4600 50  0001 C CNN
+	1    6100 4600
+	0    1    1    0
+$EndComp
+$Comp
+L power:VCC #PWR0118
+U 1 1 60BB8B38
+P 6600 4400
+F 0 "#PWR0118" H 6600 4250 50  0001 C CNN
+F 1 "VCC" V 6615 4528 50  0000 L CNN
+F 2 "" H 6600 4400 50  0001 C CNN
+F 3 "" H 6600 4400 50  0001 C CNN
+	1    6600 4400
+	0    1    1    0
+$EndComp
+Text GLabel 4900 1600 2    50   Input ~ 0
+sclk
+Text GLabel 4900 1700 2    50   Input ~ 0
+miso
+Text GLabel 4900 2600 2    50   Input ~ 0
+mosi
+Text GLabel 4900 2100 2    50   Input ~ 0
+ss
 $EndSCHEMATC

Commit message: Finished The Final Result
Gerbers and everything :DD
Connections:
- net motion: no longer names the net of J4.2 (Pin_2)
Changed lines of the file:
@@
 Text GLabel 6100 4400 0    50   Input ~ 0
 ss
-Text GLabel 6100 4500 0    50   Input ~ 0
-motion
 Text GLabel 6600 4500 2    50   Input ~ 0
 miso
