File: Productivity Macro.kicad_pcb (KiCad board)
At the start: 2 copper layers, 34 parts, among them SW1 SW_Push, SW2 Rotary_Encoder_Switch, SW3 Rotary_Encoder_Switch, U1 ATmega32U4-AU, Y1 16Mhz

Commit message: this is stupid
Connections:
- U1 pad 22: Net-(U1-Pad22) -> ROW0
- U1 pad 25: COL0 -> Net-(U1-Pad25)
- U1 pad 26: COL1 -> ROW2
- U1 pad 27: COL2 -> Net-(U1-Pad27)
- U1 pad 30: ROW2 -> Net-(U1-Pad30)
- U1 pad 31: ROW0 -> Net-(U1-Pad31)
- U1 pad 37: Net-(U1-Pad37) -> COL2
- U1 pad 38: Net-(U1-Pad38) -> COL1
- U1 pad 39: Net-(U1-Pad39) -> COL0
Routing:
- net COL2: track 39.4 -> 88.3 mm, vias 0 -> 1
- net ROW0: track 19.8 -> 49.7 mm, vias 2 -> 7
- net ROW2: track 20.5 -> 44.5 mm, vias 0 -> 1
- net COL1: track 38.1 -> 58.5 mm
- net COL0: track 40.5 -> 60.8 mm, vias 0 -> 1
- net +5V: track 161.0 -> 168.8 mm, vias 6 -> 8
- net GND: track 155.3 -> 159.6 mm, vias 2 -> 4
- net Net-(R1-Pad2): track 85.8 -> 86.6 mm
- net Net-(U1-Pad25): track 0.00 -> 0.79 mm
Other:
- board text added: "This is Stupid"
