File: Productivity Macro.kicad_pcb (KiCad board)
At the start: 2 copper layers, 35 parts, among them J4 Conn_02x04_Counter_Clockwise, SW1 SW_Push, SW2 Rotary_Encoder_Switch, SW3 Rotary_Encoder_Switch, U1 ATmega32U4-AU, Y1 16Mhz

Commit message: Finished The Final Result
Gerbers and everything :DD
Parts:
- added G***: LOGO, Revamped Graphics:The real better one, F.Cu at (207.8, 63.0)
Connections:
- net motion renamed Net-(J4-Pad2)
Routing:
- added copper zone on B.Cu, net (none)
- added copper zone on F.Cu, net (none)
Other:
- board outline added: 65.8 x 88.9 mm
- board text added: "GND"
- board text added: "MISO"
- board text added: "MOSI"
- board text added: "SCLK"
- board text added: "SS"
- board text added: "VCC"

Commit message: revamp
Routing:
- net Net-(D3-Pad2): track 13.5 -> 12.1 mm
- net +5V: track 165.7 -> 164.6 mm
- net GND: track 266.9 -> 266.1 mm
- net Net-(R1-Pad2): track 86.6 -> 85.9 mm
- net ROW2: track 44.5 -> 44.0 mm
- removed copper zone on B.Cu, net (none)
- removed copper zone on F.Cu, net (none)
