File: Productivity Macro Backup.kicad_pcb (KiCad board)
At the start: 2 copper layers, 35 parts, among them J4 Conn_02x04_Counter_Clockwise, SW1 SW_Push, SW2 Rotary_Encoder_Switch, SW3 Rotary_Encoder_Switch, U1 ATmega32U4-AU, Y1 16Mhz

Commit message: The beginning of the trackball
Parts:
- removed J4: Conn_02x04_Counter_Clockwise, Connector_PinSocket_2.00mm:PinSocket_2x04_P2.00mm_Vertical
Connections:
- U1 pad 18: mosi -> Net-(U1-Pad18)
- U1 pad 28: Net-(U1-Pad28) -> mosi
Routing:
- net VCC: track 63.2 -> 6.82 mm
- net mosi: track 54.0 -> 0.00 mm, vias 2 -> 0
- net GND: track 266.9 -> 249.5 mm, vias 9 -> 7
- net miso: track 13.7 -> 0.00 mm, vias 2 -> 0
- net ss: track 12.8 -> 0.00 mm, vias 2 -> 0
- net sclk: track 11.2 -> 0.00 mm, vias 2 -> 0
- net +5V: track 165.7 -> 168.8 mm
